File: prototipo_do_lab/primeira_camada_recepcao.kicad_sch (KiCad schematic)
At the start: 7 parts, among them J9 0732511352, U13 SKY13373-460LF

Commit message: footprint uptated in board still needs validation
Parts:
- U13: footprint SKY13373-460LF:QFN50P200X200X65-13N -> SKY13373-460LF:QFN50P200X200X65-13N_1LabProt
Changed lines of the file:
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@@
 			)
 		)
-		(property "Footprint" "SKY13373-460LF:QFN50P200X200X65-13N"
+		(property "Footprint" "SKY13373-460LF:QFN50P200X200X65-13N_1LabProt"
 			(at 144.78 95.25 0)
 			(effects
@@
 				)
 				(justify bottom)
-				(hide yes)
 			)
 		)
