File: prototipo_do_lab/segunda_camada_emissao.kicad_sch (KiCad schematic)
At the start: 19 parts, among them J10 0732511352, U2 SKY13373-460LF, U3 SKY13373-460LF, U4 SKY13373-460LF

Commit message: footprint uptated in board still needs validation
Parts:
- U2, U3, U4: footprint SKY13373-460LF:QFN50P200X200X65-13N -> SKY13373-460LF:QFN50P200X200X65-13N_1LabProt
Changed lines of the file:
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@@
 			)
 		)
-		(property "Footprint" "SKY13373-460LF:QFN50P200X200X65-13N"
+		(property "Footprint" "SKY13373-460LF:QFN50P200X200X65-13N_1LabProt"
 			(at 129.54 125.73 0)
 			(effects
@@
 			)
 		)
-		(property "Footprint" "SKY13373-460LF:QFN50P200X200X65-13N"
+		(property "Footprint" "SKY13373-460LF:QFN50P200X200X65-13N_1LabProt"
 			(at 129.54 91.44 0)
 			(effects
@@
 			)
 		)
-		(property "Footprint" "SKY13373-460LF:QFN50P200X200X65-13N"
+		(property "Footprint" "SKY13373-460LF:QFN50P200X200X65-13N_1LabProt"
 			(at 129.54 57.15 0)
 			(effects
