File: EVAL_TRILHA_V2/eval_trilha_v2/eval_trilha_v2.kicad_pcb (KiCad board)
At the start: 4 copper layers, 100 x 100 mm, 27 parts, among them J0 0732511352, J1 0732511352, J10 0732511352, J11 0732511352, J12 TSW-205-14-L-S, J13 0732511352, J14 0732511352, J15 0732511352, J16 0732511352, J17 CON-SMA-EDGE-S, J18 CON-SMA-EDGE-S, J2 0732511352, J3 0732511352, J4 0732511352, J5 0732511352, J6 0732511352, J7 0732511352, J8 0732511352, J9 0732511352, U1 SKY13373-460LF

Commit message: feat(eval): track W updated to lauquen specifications, still need to update the board stackup
Routing:
- net GND: track 0.00 -> 8.04 mm, vias 376 -> 379
Other:
- board text added: "0.240mm"
- board text added: "0.254mm"
- board text added: "0.254mm Manufacturer Suggestion (10 Mils)"
- board text added: "0.254mm Sugestion"
- board text added: "0.271mm Calculated with KiCad"
- board text added: "0.308mm Calculated with KiCad"

Commit message: track width up to date on lauquen recommendation
Other:
- board text added: "0.291mm Calculated with KiCad"
- board text removed: "0.308mm Calculated with KiCad"
Changed lines of the file:
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@@
 	(generator_version "9.0")
 	(general
-		(thickness 1.6)
+		(thickness 1.584)
 		(legacy_teardrops no)
 	)
@@
 			(layer "F.Mask"
 				(type "Top Solder Mask")
-				(thickness 0.01)
+				(thickness 0.025)
 			)
 			(layer "F.Cu"
 				(type "copper")
-				(thickness 0.035)
+				(thickness 0.017)
 			)
 			(layer "dielectric 1"
 				(type "prepreg")
-				(thickness 0.1)
+				(thickness 0.15)
 				(material "FR4")
 				(epsilon_r 4.5)
@@
 			(layer "dielectric 2"
 				(type "core")
-				(thickness 1.24)
+				(thickness 1.13)
 				(material "FR4")
 				(epsilon_r 4.5)
@@
 			(layer "dielectric 3"
 				(type "prepreg")
-				(thickness 0.1)
+				(thickness 0.15)
 				(material "FR4")
 				(epsilon_r 4.5)
@@
 			(layer "B.Cu"
 				(type "copper")
-				(thickness 0.035)
+				(thickness 0.017)
 			)
 			(layer "B.Mask"
 				(type "Bottom Solder Mask")
-				(thickness 0.01)
+				(thickness 0.025)
 			)
 			(layer "B.Paste"
@@
 		)
 	)
-	(gr_text "0.308mm Calculated with KiCad"
+	(gr_text "0.291mm Calculated with KiCad"
 		(at 167 57.96 0)
 		(layer "F.SilkS")
@@
 		)
 	)
-	(gr_text "0.308mm Calculated with KiCad"
+	(gr_text "0.291mm Calculated with KiCad"
 		(at 122 105.5 0)
 		(layer "F.SilkS")
@@
 		(start 191 105.953056)
 		(end 111.25 105.953056)
-		(width 0.308)
+		(width 0.291)
 		(layer "F.Cu")
 		(net 0)
@@
 		(start 191 58.328611)
 		(end 161.25 58.328611)
-		(width 0.308)
+		(width 0.291)
 		(layer "F.Cu")
 		(net 7)
