File: MATRIZ_DE_CHAVEAMENTO/untitled.kicad_sch (KiCad schematic)
At the start: 64 parts, among them J1 0732511352, J12 0732511352, J2 0732511352, J3 0732511352, J4 0732511352, J5 0732511352, J6 0732511352, J7 0732511352, U10 SKY13373-460LF, U11 SKY13373-460LF, U12 SKY13373-460LF, U5 SKY13373-460LF, U6 SKY13373-460LF, U7 SKY13373-460LF, U8 SKY13373-460LF, U9 SKY13373-460LF

Commit message: footprint correction ongoing
Parts:
- U9: footprint SKY13373-460LF:QFN50P200X200X65-13N_1LabProt -> SKY13373-460LF:QFN50P200X200X65-13N
Changed lines of the file:
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@@
 			)
 		)
-		(property "Footprint" "SKY13373-460LF:QFN50P200X200X65-13N_1LabProt"
+		(property "Footprint" "SKY13373-460LF:QFN50P200X200X65-13N"
 			(at 152.4 96.52 0)
 			(effects

Commit message: footprint up to date
Parts:
- U10, U11, U12, U5, U6, U7, U8: footprint SKY13373-460LF:QFN50P200X200X65-13N_1LabProt -> SKY13373-460LF:QFN50P200X200X65-13N
Changed lines of the file:
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@@
 			)
 		)
-		(property "Footprint" "SKY13373-460LF:QFN50P200X200X65-13N_1LabProt"
+		(property "Footprint" "SKY13373-460LF:QFN50P200X200X65-13N"
 			(at 152.4 130.81 0)
 			(effects
@@
 			)
 		)
-		(property "Footprint" "SKY13373-460LF:QFN50P200X200X65-13N_1LabProt"
+		(property "Footprint" "SKY13373-460LF:QFN50P200X200X65-13N"
 			(at 64.77 130.81 0)
 			(effects
@@
 			)
 		)
-		(property "Footprint" "SKY13373-460LF:QFN50P200X200X65-13N_1LabProt"
+		(property "Footprint" "SKY13373-460LF:QFN50P200X200X65-13N"
 			(at 152.4 62.23 0)
 			(effects
@@
 			)
 		)
-		(property "Footprint" "SKY13373-460LF:QFN50P200X200X65-13N_1LabProt"
+		(property "Footprint" "SKY13373-460LF:QFN50P200X200X65-13N"
 			(at 64.77 96.52 0)
 			(effects
@@
 			)
 		)
-		(property "Footprint" "SKY13373-460LF:QFN50P200X200X65-13N_1LabProt"
+		(property "Footprint" "SKY13373-460LF:QFN50P200X200X65-13N"
 			(at 64.77 62.23 0)
 			(effects
@@
 			)
 		)
-		(property "Footprint" "SKY13373-460LF:QFN50P200X200X65-13N_1LabProt"
+		(property "Footprint" "SKY13373-460LF:QFN50P200X200X65-13N"
 			(at 240.03 96.52 0)
 			(effects
@@
 			)
 		)
-		(property "Footprint" "SKY13373-460LF:QFN50P200X200X65-13N_1LabProt"
+		(property "Footprint" "SKY13373-460LF:QFN50P200X200X65-13N"
 			(at 240.03 62.23 0)
 			(effects

Commit message: feat(footprint): RF switch footprint updated
Parts:
- U10, U11, U12, U5, U6, U7, U8, U9: footprint SKY13373-460LF:QFN50P200X200X65-13N -> SKY13373-460LF:QFN50P200X200X65-13N_1LabProt
Changed lines of the file:
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@@
 			)
 		)
-		(property "Footprint" "SKY13373-460LF:QFN50P200X200X65-13N"
+		(property "Footprint" "SKY13373-460LF:QFN50P200X200X65-13N_1LabProt"
 			(at 152.4 130.81 0)
 			(effects
@@
 			)
 		)
-		(property "Footprint" "SKY13373-460LF:QFN50P200X200X65-13N"
+		(property "Footprint" "SKY13373-460LF:QFN50P200X200X65-13N_1LabProt"
 			(at 64.77 130.81 0)
 			(effects
@@
 			)
 		)
-		(property "Footprint" "SKY13373-460LF:QFN50P200X200X65-13N"
+		(property "Footprint" "SKY13373-460LF:QFN50P200X200X65-13N_1LabProt"
 			(at 152.4 62.23 0)
 			(effects
@@
 			)
 		)
-		(property "Footprint" "SKY13373-460LF:QFN50P200X200X65-13N"
+		(property "Footprint" "SKY13373-460LF:QFN50P200X200X65-13N_1LabProt"
 			(at 64.77 96.52 0)
 			(effects
@@
 			)
 		)
-		(property "Footprint" "SKY13373-460LF:QFN50P200X200X65-13N"
+		(property "Footprint" "SKY13373-460LF:QFN50P200X200X65-13N_1LabProt"
 			(at 64.77 62.23 0)
 			(effects
@@
 			)
 		)
-		(property "Footprint" "SKY13373-460LF:QFN50P200X200X65-13N"
+		(property "Footprint" "SKY13373-460LF:QFN50P200X200X65-13N_1LabProt"
 			(at 152.4 96.52 0)
 			(effects
@@
 			)
 		)
-		(property "Footprint" "SKY13373-460LF:QFN50P200X200X65-13N"
+		(property "Footprint" "SKY13373-460LF:QFN50P200X200X65-13N_1LabProt"
 			(at 240.03 96.52 0)
 			(effects
@@
 			)
 		)
-		(property "Footprint" "SKY13373-460LF:QFN50P200X200X65-13N"
+		(property "Footprint" "SKY13373-460LF:QFN50P200X200X65-13N_1LabProt"
 			(at 240.03 62.23 0)
 			(effects
