File: MATRIZ_DE_CHAVEAMENTO/Imageamento_microondas.kicad_pcb (KiCad board)
At the start: 4 copper layers, 200 x 150 mm, 121 parts, among them J1 0732511352, J10 0732511352, J11 TB0012-508-03GR, J12 0732511352, J13 0732511352, J2 0732511352, J3 0732511352, J4 0732511352, J5 0732511352, J6 0732511352, J7 0732511352, J8 0732511352, J9 0732511352, U1 SKY13373-460LF, U10 SKY13373-460LF, U11 SKY13373-460LF, U12 SKY13373-460LF, U13 SKY13373-460LF, U14 SKY13373-460LF, U15 SKY13373-460LF, U16 SKY13373-460LF, U17 ESP32-DEVKITC-32E, U18 MCP23016-I_SP, U2 SKY13373-460LF, U3 SKY13373-460LF, U4 SKY13373-460LF, U5 SKY13373-460LF, U6 SKY13373-460LF, U7 SKY13373-460LF, U8 SKY13373-460LF, U9 SKY13373-460LF

Commit message: eval added to main board, still incomplete
Parts:
- added C49: C, Capacitor_SMD:C_0402_1005Metric, F.Cu at (121.8, 156.4)
- added C51: C, Capacitor_SMD:C_0402_1005Metric, F.Cu at (125.5, 156.5)
- added C52: C, Capacitor_SMD:C_0402_1005Metric, F.Cu at (129.2, 156.5)
- added J14: 0732511352, conector_sma:Footprint_adaptado, F.Cu at (197.3, 157.3)
- added J15: 0732511352, conector_sma:Footprint_adaptado, F.Cu at (156.2, 157.3)
- added J16: 0732511352, conector_sma:Footprint_adaptado, F.Cu at (115.1, 137.8)
- added J17: 0732511352, conector_sma:Footprint_adaptado, F.Cu at (104.2, 148.6)
- added J18: 0732511352, conector_sma:Footprint_adaptado, F.Cu at (115.1, 159.4)
- added J19: 0732511352, conector_sma:Footprint_adaptado, F.Cu at (126.0, 148.6)
- added U19: SKY13373-460LF, SKY13373-460LF:QFN50P200X200X65-13N, F.Cu at (115.3, 148.6)
- U1, U10, U11, U12, U13, U14, U15, U16, U2, U3, U4, U5, U6, U7, U8, U9: footprint SKY13373-460LF:QFN50P200X200X65-13N -> SKY13373-460LF:QFN50P200X200X65-13N_1LabProt
Routing:
- net Net-(J14-Pad1): track 0.00 -> 40.8 mm
- net /arbitragem/T3: track 0.00 -> 10.4 mm
- net /arbitragem/T1: track 0.00 -> 10.2 mm
- net /arbitragem/T2: track 0.00 -> 9.72 mm
- net Net-(U19-RFC): track 0.00 -> 9.70 mm
- net GND: vias 2258 -> 2254

Commit message: finished eval on main board
Parts:
- added J20: 0732511352, conector_sma:Footprint_adaptado, F.Cu at (153.9, 143.7)
- added J21: 0732511352, conector_sma:Footprint_adaptado, F.Cu at (176.1, 143.7)
- added TP33: TestPoint, TestPoint:TestPoint_Pad_D1.5mm, B.Cu at (112.6, 145.6)
- added TP34: TestPoint, TestPoint:TestPoint_Pad_D1.5mm, B.Cu at (117.7, 145.6)
- moved C52 7.05 mm to (122.5, 154.6)
- moved C51 6.06 mm to (120.2, 153.6)
- moved C49 5.63 mm to (116.9, 153.6)
- moved J15 2.33 mm to (153.9, 157.3)
- moved J14 1.25 mm to (196.1, 157.3)
Routing:
- net Net-(J20-Pad1): track 0.00 -> 21.0 mm
- net /arbitragem/Ctrl2: track 0.00 -> 15.0 mm, vias 0 -> 1
- net /arbitragem/Ctrl1: track 0.00 -> 13.7 mm, vias 0 -> 1
- net VDD: track 80.0 -> 91.9 mm, vias 16 -> 17
- net Net-(J14-Pad1): track 40.8 -> 40.0 mm
- net GND: vias 2254 -> 2252
