File: MATRIZ_DE_CHAVEAMENTO/Imageamento_microondas.kicad_pcb (KiCad board)
At the start: 4 copper layers, 200 x 150 mm, 135 parts, among them J1 0732511352, J10 0732511352, J11 TB0012-508-03GR, J12 0732511352, J13 0732511352, J14 0732511352, J15 0732511352, J16 0732511352, J17 0732511352, J18 0732511352, J19 0732511352, J2 0732511352, J20 0732511352, J21 0732511352, J3 0732511352, J4 0732511352, J5 0732511352, J6 0732511352, J7 0732511352, J8 0732511352, J9 0732511352, U1 SKY13373-460LF, U10 SKY13373-460LF, U11 SKY13373-460LF, U12 SKY13373-460LF, U13 SKY13373-460LF, U14 SKY13373-460LF, U15 SKY13373-460LF, U16 SKY13373-460LF, U17 ESP32-DEVKITC-32E, U18 MCP23016-I_SP, U19 SKY13373-460LF, U2 SKY13373-460LF, U3 SKY13373-460LF, U4 SKY13373-460LF, U5 SKY13373-460LF, U6 SKY13373-460LF, U7 SKY13373-460LF, U8 SKY13373-460LF, U9 SKY13373-460LF

Commit message: footprint correction ongoing
Parts:
- U9: footprint SKY13373-460LF:QFN50P200X200X65-13N_1LabProt -> SKY13373-460LF:QFN50P200X200X65-13N
- moved C27 0.81 mm to (84.2, 96.5), turned to 90 degrees
- moved C33 0.76 mm to (157.1, 82.0), turned to 90 degrees
- moved C41 0.75 mm to (218.7, 123.4), turned to 90 degrees
Routing:
- net GND: track 0.00 -> 165.7 mm, vias 2252 -> 2305
- net VDD: track 91.9 -> 96.5 mm
- net Net-(U5-RFC): track 14.2 -> 11.4 mm
- net Net-(U10-RFC): track 14.2 -> 11.5 mm
- net Net-(U9-RFC): track 14.4 -> 16.6 mm
- net Net-(U12-RFC): track 14.5 -> 13.6 mm
- net Net-(U8-RFC): track 14.3 -> 14.8 mm
- net /CE2_1: track 153.8 -> 154.3 mm

Commit message: footprint up to date
Parts:
- U1, U10, U11, U12, U13, U14, U15, U16, U2, U3, U4, U5, U6, U7, U8: footprint SKY13373-460LF:QFN50P200X200X65-13N_1LabProt -> SKY13373-460LF:QFN50P200X200X65-13N
Connections:
- U19 pad 10: Net-(U19-GND-Pad10) -> GND
- U19 pad 12: Net-(U19-GND-Pad10) -> GND
- U19 pad 13: Net-(U19-GND-Pad10) -> GND
- U19 pad 2: Net-(U19-GND-Pad10) -> GND
- U19 pad 7: Net-(U19-GND-Pad10) -> GND
- U19 pad 8: Net-(U19-GND-Pad10) -> GND
Routing:
- net GND: track 165.7 -> 300.4 mm, vias 2305 -> 2309
