File: MATRIZ_DE_CHAVEAMENTO/arbitragem.kicad_sch (KiCad schematic)
At the start: 5 parts, among them J11 TB0012-508-03GR, U17 ESP32-DEVKITC-32E, U18 MCP23016-I_SP

Commit message: eval added to main board, still incomplete
Parts:
- added C49, C51, C52: C, Capacitor_SMD:C_0402_1005Metric, symbol Device:C
- added J14, J15, J16, J17, J18, J19: 0732511352, conector_sma:Footprint_adaptado, symbol 0732511352:0732511352
- added U19: SKY13373-460LF, SKY13373-460LF:QFN50P200X200X65-13N, symbol SKY13373-460LF:SKY13373-460LF
Connections:
- net GND: now also C49.1, C51.2, C52.2, J14.S1, J14.S2, J14.S3, J14.S4, J15.S1, J15.S2, J15.S3, J15.S4, J16.S1, J16.S2, J16.S3, J16.S4, J17.S1, J17.S2, J17.S3, J17.S4, J18.S1, J18.S2, J18.S3, J18.S4, J19.S1, J19.S2, J19.S3, J19.S4
- net VDD: now also C52.1, U19.6 (VDD)
- new net: U19.10 (GND), U19.12 (GND), U19.13 (GND), U19.2 (GND), U19.7 (GND), U19.8 (GND)
- new net: J16.1, U19.11 (RFC)
- new net: J14.1, J15.1
- new net Ctrl1: C49.2, U19.4 (V1)
- new net Ctrl2: C51.1, U19.5 (V2)
- new net T1: J17.1, U19.1 (J1)
- new net T2: J19.1, U19.9 (J2)
- new net T3: J18.1, U19.3 (J3)
Other:
- moved on the sheet: C50, R9, U18

Commit message: finished eval on main board
Parts:
- added J20, J21: 0732511352, conector_sma:Footprint_adaptado, symbol 0732511352:0732511352
- added TP33, TP34: TestPoint, TestPoint:TestPoint_Pad_D1.5mm, symbol Connector:TestPoint
Connections:
- net Ctrl1: now also TP33.1
- net Ctrl2: now also TP34.1
- net GND: now also J20.S1, J20.S2, J20.S3, J20.S4, J21.S1, J21.S2, J21.S3, J21.S4
- new net: J20.1, J21.1

Commit message: footprint up to date
Connections:
- net GND: now also U19.10 (GND), U19.12 (GND), U19.13 (GND), U19.2 (GND), U19.7 (GND), U19.8 (GND)
Changed lines of the file:
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@@
 		)
 	)
+	(wire
+		(pts
+			(xy 259.08 77.47) (xy 259.08 74.93)
+		)
+		(stroke
+			(width 0)
+			(type default)
+		)
+	)
 	(bus
 		(pts
@@
 					(unit 1)
 				)
+			)
+		)
+	)
+	(symbol
+		(lib_id "power:GND")
+		(at 259.08 77.47 0)
+		(unit 1)
+		(exclude_from_sim no)
+		(in_bom yes)
+		(on_board yes)
+		(dnp no)
+		(fields_autoplaced yes)
+		(property "Reference" "#PWR0121"
+			(at 259.08 83.82 0)
+			(effects
+				(font
+					(size 1.27 1.27)
+				)
+				(hide yes)
+			)
+		)
+		(property "Value" "GND"
+			(at 259.08 82.55 0)
+			(effects
+				(font
+					(size 1.27 1.27)
+				)
+			)
+		)
+		(property "Footprint" ""
+			(at 259.08 77.47 0)
+			(effects
+				(font
+					(size 1.27 1.27)
+				)
+				(hide yes)
+			)
+		)
+		(property "Datasheet" ""
+			(at 259.08 77.47 0)
+			(effects
+				(font
+					(size 1.27 1.27)
+				)
+				(hide yes)
+			)
+		)
+		(property "Description" "Power symbol creates a global label with name \"GND\" , ground"
+			(at 259.08 77.47 0)
+			(effects
+				(font
+					(size 1.27 1.27)
+				)
+				(hide yes)
+			)
+		)
+		(pin "1"
+		)
+		(instances
+			(project "Imageamento_microondas"
+				(path "/cdf0ef36-17ab-4910-af08-9c79f1680f36/94333ec5-1b9c-4318-b308-51cf4235b858"
+					(reference "#PWR0121")
+					(unit 1)
+				)
