File: MATRIZ_DE_CHAVEAMENTO/primeira_camada_emissao.kicad_sch (KiCad schematic)
At the start: 7 parts, among them J8 0732511352, U1 SKY13373-460LF

Commit message: feat(footprint): RF switch footprint updated
Parts:
- U1: footprint SKY13373-460LF:QFN50P200X200X65-13N -> SKY13373-460LF:QFN50P200X200X65-13N_1LabProt
Changed lines of the file:
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@@
 			)
 		)
-		(property "Footprint" "SKY13373-460LF:QFN50P200X200X65-13N"
+		(property "Footprint" "SKY13373-460LF:QFN50P200X200X65-13N_1LabProt"
 			(at 142.24 100.33 0)
 			(effects

Commit message: footprint up to date
Parts:
- U1: footprint SKY13373-460LF:QFN50P200X200X65-13N_1LabProt -> SKY13373-460LF:QFN50P200X200X65-13N
Changed lines of the file:
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@@
 			)
 		)
-		(property "Footprint" "SKY13373-460LF:QFN50P200X200X65-13N_1LabProt"
+		(property "Footprint" "SKY13373-460LF:QFN50P200X200X65-13N"
 			(at 142.24 100.33 0)
 			(effects
