File: MATRIZ_DE_CHAVEAMENTO/segunda_camada_emissao.kicad_sch (KiCad schematic)
At the start: 19 parts, among them J10 0732511352, U2 SKY13373-460LF, U3 SKY13373-460LF, U4 SKY13373-460LF

Commit message: feat(footprint): RF switch footprint updated
Parts:
- U2, U3, U4: footprint SKY13373-460LF:QFN50P200X200X65-13N -> SKY13373-460LF:QFN50P200X200X65-13N_1LabProt
Changed lines of the file:
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@@
 	)
 	(bus_entry
+		(at 203.2 100.33)
+		(size 2.54 2.54)
+		(stroke
+			(width 0)
+			(type default)
+		)
+	)
+	(bus_entry
 		(at 82.55 138.43)
 		(size 2.54 2.54)
@@
 			)
 		)
-		(property "Footprint" "SKY13373-460LF:QFN50P200X200X65-13N"
+		(property "Footprint" "SKY13373-460LF:QFN50P200X200X65-13N_1LabProt"
 			(at 129.54 125.73 0)
 			(effects
@@
 			)
 		)
-		(property "Footprint" "SKY13373-460LF:QFN50P200X200X65-13N"
+		(property "Footprint" "SKY13373-460LF:QFN50P200X200X65-13N_1LabProt"
 			(at 129.54 91.44 0)
 			(effects
@@
 			)
 		)
-		(property "Footprint" "SKY13373-460LF:QFN50P200X200X65-13N"
+		(property "Footprint" "SKY13373-460LF:QFN50P200X200X65-13N_1LabProt"
 			(at 129.54 57.15 0)
 			(effects

Commit message: footprint up to date
Parts:
- U2, U3, U4: footprint SKY13373-460LF:QFN50P200X200X65-13N_1LabProt -> SKY13373-460LF:QFN50P200X200X65-13N
Changed lines of the file:
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@@
 			)
 		)
-		(property "Footprint" "SKY13373-460LF:QFN50P200X200X65-13N_1LabProt"
+		(property "Footprint" "SKY13373-460LF:QFN50P200X200X65-13N"
 			(at 129.54 125.73 0)
 			(effects
@@
 			)
 		)
-		(property "Footprint" "SKY13373-460LF:QFN50P200X200X65-13N_1LabProt"
+		(property "Footprint" "SKY13373-460LF:QFN50P200X200X65-13N"
 			(at 129.54 91.44 0)
 			(effects
@@
 			)
 		)
-		(property "Footprint" "SKY13373-460LF:QFN50P200X200X65-13N_1LabProt"
+		(property "Footprint" "SKY13373-460LF:QFN50P200X200X65-13N"
 			(at 129.54 57.15 0)
 			(effects
